File: pcb/Arduino Shield/Arduino Shield.kicad_pcb (KiCad board)
At the start: 2 copper layers, 101.6 x 53.3 mm, 47 parts, among them J1 Power, J10 CH_02, J11 CH_03, J12 CH_04, J13 CH_05, J14 Main Controller, J15 DRV_03, J16 DRV_02, J17 DRV_01, J18 EXT VCC, J19 DRV_03_PWR, J2 PWM, J20 SD_SPI, J21 DRV_02_PWR, J22 DRV_01_PWR, J23 Panel Power SW, J3 Analog, J4 PWM, J5 Analog, J6 Communication, J7 Digital, J8 SCR_SPI, J9 CH_01

Commit message: Silkscreen updates.
Parts:
- J23: value Panel Power SW -> Panel PSW
Routing:
- net (no net): track 4302.9 -> 0.00 mm
