File: pcb/Teensy (V2)/Teensy Version.kicad_pcb (KiCad board)
At the start: 2 copper layers, 30 parts, among them J1 DRV_01, J10 CH_02, J11 CH_03, J12 CH_04, J13 CH_05, J14 Main Controller, J18 EXT VCC, J2 DRV_02, J23 Panel Power SW, J3 DRV_03, J4 DRV_05, J5 DRV_04, J8 SCR_SPI, J9 CH_01, U1 Teensy4.1, U2 74HC138, U4 74HC595, U5 MCP23017_SO

Commit message: Fix up channel pcb
Parts:
- removed U4: 74HC595, Package_SO:SO-16_3.9x9.9mm_P1.27mm
- added U3: MCP23017_SO, Package_SO:SOIC-28W_7.5x17.9mm_P1.27mm, F.Cu at (90.5, 72.9)
- moved D1 61.3 mm to (130.1, 80.5)
- moved R1 57.6 mm to (133.3, 97.5)
- moved U2 54.4 mm to (136.0, 89.8)
- moved U5 40.3 mm to (103.4, 72.9)
- moved J8 38.0 mm to (106.3, 84.7)
- moved C10 24.8 mm to (111.4, 69.1)
- moved C11 24.8 mm to (111.4, 73.2)
- moved C12 24.8 mm to (111.4, 77.2)
- moved C14 24.8 mm to (111.4, 85.3)
- moved C15 24.8 mm to (111.4, 89.4)
- moved C9 24.8 mm to (111.4, 65.1)
- moved J18 24.8 mm to (140.2, 65.1)
- moved J23 24.8 mm to (144.3, 65.1)
- moved J4 24.8 mm to (132.2, 65.1)
- moved F1 24.8 mm to (120.1, 73.1)
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Connections:
- U1 pad 14: SCR_DC_LATCH -> unconnected-(U1-12_MISO_MQSL-Pad14)
- U1 pad 25: CH4_MOTOR_A -> CH1_SCR_DC
- U1 pad 26: CH4_MOTOR_B -> CH2_SCR_DC
- U1 pad 27: CH5_MOTOR_A -> CH3_SCR_DC
- U1 pad 28: CH5_MOTOR_B -> CH4_SCR_DC
- U1 pad 31: unconnected-(U1-39_MISO1_OUT1A-Pad31) -> CH5_SCR_DC
- U1 pad 32: unconnected-(U1-40_A16-Pad32) -> CH_MAIN_SCR_DC
- U1 pad 40: CH1_MOTOR_A -> unconnected-(U1-18_A4_SDA-Pad40)
- U1 pad 41: CH1_MOTOR_B -> unconnected-(U1-19_A5_SCL-Pad41)
- U1 pad 42: CH2_MOTOR_A -> unconnected-(U1-20_A6_TX5_LRCLK1-Pad42)
- U1 pad 43: CH2_MOTOR_B -> unconnected-(U1-21_A7_RX5_BCLK1-Pad43)
- U1 pad 44: CH3_MOTOR_A -> unconnected-(U1-22_A8_CTX1-Pad44)
- U1 pad 45: CH3_MOTOR_B -> unconnected-(U1-23_A9_CRX1_MCLK1-Pad45)
