File: pcb/Teensy (V2)/Teensy Version.kicad_sch (KiCad schematic)
At the start: 30 parts, among them J1 DRV_01, J10 CH_02, J11 CH_03, J12 CH_04, J13 CH_05, J14 Main Controller, J18 EXT VCC, J2 DRV_02, J23 Panel Power SW, J3 DRV_03, J4 DRV_05, J5 DRV_04, J8 SCR_SPI, J9 CH_01, U1 Teensy4.1, U2 74HC138, U4 74HC595, U5 MCP23017_SO

Commit message: Fix up channel pcb
Parts:
- removed U4: 74HC595, Package_SO:SO-16_3.9x9.9mm_P1.27mm, symbol 74xx:74HC595
- added U3: MCP23017_SO, Package_SO:SOIC-28W_7.5x17.9mm_P1.27mm, symbol Interface_Expansion:MCP23017_SO
Connections:
- net 3v3: now also U3.15 (A0), U3.18 (~{RESET}), U3.9 (VDD)
- net CH1_MOTOR_A: now also U3.2 (GPB1); no longer U1.40 (18_A4_SDA)
- net CH1_MOTOR_B: now also U3.1 (GPB0); no longer U1.41 (19_A5_SCL)
- net CH1_SCR_DC: now also U1.25 (33_MCLK2)
- net CH2_MOTOR_A: now also U3.4 (GPB3); no longer U1.42 (20_A6_TX5_LRCLK1)
- net CH2_MOTOR_B: now also U3.3 (GPB2); no longer U1.43 (21_A7_RX5_BCLK1)
- net CH2_SCR_DC: now also U1.26 (34_RX8)
- net CH3_MOTOR_A: now also U3.6 (GPB5); no longer U1.44 (22_A8_CTX1)
- net CH3_MOTOR_B: now also U3.5 (GPB4); no longer U1.45 (23_A9_CRX1_MCLK1)
- net CH3_SCR_DC: now also U1.27 (35_TX8)
- net CH4_MOTOR_A: now also U3.8 (GPB7); no longer U1.25 (33_MCLK2)
- net CH4_MOTOR_B: now also U3.7 (GPB6); no longer U1.26 (34_RX8)
- net CH4_SCR_DC: now also U1.28 (36_CS)
- net CH5_MOTOR_A: now also U3.22 (GPA1); no longer U1.27 (35_TX8)
- net CH5_MOTOR_B: now also U3.21 (GPA0); no longer U1.28 (36_CS)
- net CH5_SCR_DC: now also U1.31 (39_MISO1_OUT1A)
- net CH_MAIN_SCR_DC: now also U1.32 (40_A16)
- net GND: now also U3.10 (VSS), U3.16 (A1), U3.17 (A2)
- net I2C_SCL: now also U3.12 (SCK)
- net I2C_SDA: now also U3.13 (SDA)
- net SCR_DC_LATCH: no longer names the net of U1.14 (12_MISO_MQSL)
- no-connect marks 19 -> 32
Other:
- moved on the sheet: C1, C2, D1, F1, J18, J23, R1
